File: eagle/schem_SMS-dumper_low.brd (EAGLE design)
At the start: 118.7 x 61 mm, 11 parts, among them IC2 74273, IC3 74273

Commit message: Add files via upload
Parts:
- removed LED: (no value), led:LED5MM
- added LD1: (no value), led:DUOLED-C-5MM
- moved R1 0.95 mm to (-28.6, 28.3)
- moved C1 0.32 mm to (-21.6, 33.3)
Connections:
- new net M0-7: IC1.34, U$1.A20
- net A15: no longer U$1.A20
- net GND: no longer LED.K
- net N$1: now also LD1.AX; no longer LED.A
- net WE: now also LD1.AR
Routing:
- net M0-7: track 0.00 -> 93.9 mm, vias 0 -> 3
- net WE: track 47.9 -> 118.0 mm, vias 0 -> 1
- net A15: track 99.6 -> 59.0 mm, vias 1 -> 0
- net GND: track 159.2 -> 134.6 mm
- net A13: track 40.4 -> 45.5 mm
- net MREQ: track 86.3 -> 89.2 mm
- net +5V: track 251.5 -> 253.9 mm
- net N$1: track 4.76 -> 3.18 mm
- net A9: track 38.9 -> 37.5 mm, vias 1 -> 0
- net D0: track 160.7 -> 162.0 mm
- net CLOCK: track 162.3 -> 161.7 mm
Other:
- board text added: "Duo led Common C 5mm"
- board text added: "v0.99 (c)2017 ICHIGO"
- board text removed: "green 5mm"
- board text removed: "v0a (c)2016 ICHIGO"
